File: 30pinsimm.kicad_pcb (KiCad board)
At the start: 4 copper layers, 89 x 16.6 mm, 7 parts, among them U1 4Mx4FPMDRAM, U2 4Mx4FPMDRAM, U3 4Mx1FPMDRAM

Commit message: updates
Other:
- board text added: "22"
- board text added: "9"

Commit message: Update 30pinsimm.kicad_pcb
Routing:
- net GND: track 27.7 -> 27.0 mm
Changed lines of the file:
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@@
     (thickness 1.2)
     (drawings 18)
-    (tracks 717)
+    (tracks 715)
     (zones 0)
     (modules 7)
@@
   (segment (start 131.9877 101.139) (end 131.9877 101.9466) (width 0.25) (layer F.Cu) (net 11))
   (segment (start 151.638 95.3798) (end 151.6888 95.329) (width 0.25) (layer F.Cu) (net 11))
-  (segment (start 161.036 97.155) (end 161.036 95.8297) (width 0.25) (layer F.Cu) (net 11))
   (segment (start 134.112 99.965) (end 133.1617 99.965) (width 0.25) (layer F.Cu) (net 11))
   (via (at 136.525 98.8707) (size 0.8) (drill 0.4) (layers F.Cu B.Cu) (net 11))
-  (via (at 160.0874 95.4462) (size 0.8) (drill 0.4) (layers F.Cu B.Cu) (net 11))
+  (via (at 161.036 95.4462) (size 0.8) (drill 0.4) (layers F.Cu B.Cu) (net 11))
   (via (at 151.638 95.377) (size 0.8) (drill 0.4) (layers F.Cu B.Cu) (net 11))
   (via (at 141.478 95.4062) (size 0.8) (drill 0.4) (layers F.Cu B.Cu) (net 11))
@@
   (segment (start 177.943 99.711) (end 177.927 99.695) (width 0.25) (layer F.Cu) (net 11))
   (segment (start 179.705 99.711) (end 177.943 99.711) (width 0.25) (layer F.Cu) (net 11))
-  (segment (start 160.6525 95.4462) (end 161.036 95.8297) (width 0.25) (layer F.Cu) (net 11))
-  (segment (start 160.0874 95.4462) (end 160.6525 95.4462) (width 0.25) (layer F.Cu) (net 11))
+  (segment (start 161.036 97.155) (end 161.036 95.4462) (width 0.25) (layer F.Cu) (net 11))
   (segment (start 153.8937 96.6912) (end 153.6186 96.9663) (width 0.25) (layer B.Cu) (net 12))
   (segment (start 153.6186 96.9663) (end 145.7849 96.9663) (width 0.25) (layer B.Cu) (net 12))

Commit message: Update 30pinsimm.kicad_pcb
Parts:
- renumbered SIMM1 to SIMM30
Changed lines of the file:
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@@
   (module Sebs:30pinSIMM (layer F.Cu)
     (at 99.441 111.379)
-    (fp_text reference SIMM1 (at 85.725 -14.224 180) (layer F.SilkS)
+    (fp_text reference SIMM30 (at 84.963 -14.351 180) (layer F.SilkS)
       (effects (font (size 1 1) (thickness 0.15)))
     )
