File: 30pinsimm.kicad_pcb (KiCad board)
At the start: 4 copper layers, 89 x 16.6 mm, 7 parts, among them U1 4Mx4FPMDRAM, U2 4Mx4FPMDRAM, U3 4Mx1FPMDRAM

Commit message: issue version 1.0
Other:
- board text added: "4MB SIMM"
- board text added: "v1.0"
- board text removed: "4Mb"
